File: vortex-f1-d-clone.kicad_pcb (KiCad board)
At the start: 2 copper layers, 39 parts, among them IC01 74LS136, IC02 74LS74, IC03 74LS85, IC04 27128, IC05 74LS14, IC06 74LS08, IC07 74LS25, IC08 74LS32, IC09 FDC_9229, IC10 uPD765AC, IC11 74LS01, IC12 74LS38, IC13 74LS07, IC14 74LS139

Commit message: PCB work
Parts:
- removed RN1: 10k, Resistor_THT:R_Array_SIP9
- added C1: 100n, Capacitor_SMD:C_0603_1608Metric_Pad1.08x0.95mm_HandSolder, F.Cu at (132.6, 73.2)
- added C11: 100n, Capacitor_SMD:C_0603_1608Metric_Pad1.08x0.95mm_HandSolder, F.Cu at (132.6, 55.4)
- added C12: 100n, Capacitor_SMD:C_0603_1608Metric_Pad1.08x0.95mm_HandSolder, F.Cu at (107.2, 85.9)
- added C14: 100n, Capacitor_SMD:C_0603_1608Metric_Pad1.08x0.95mm_HandSolder, F.Cu at (73.2, 97.2)
- added C15: 100n, Capacitor_SMD:C_0603_1608Metric_Pad1.08x0.95mm_HandSolder, F.Cu at (88.4, 59.9)
- added C16: 100n, Capacitor_SMD:C_0603_1608Metric_Pad1.08x0.95mm_HandSolder, F.Cu at (27.4, 73.2)
- added C17: 100n, Capacitor_SMD:C_0603_1608Metric_Pad1.08x0.95mm_HandSolder, F.Cu at (27.4, 35.1)
- added C2: 100n, Capacitor_SMD:C_0603_1608Metric_Pad1.08x0.95mm_HandSolder, F.Cu at (55.4, 35.1)
- added C3: 100n, Capacitor_SMD:C_0603_1608Metric_Pad1.08x0.95mm_HandSolder, F.Cu at (55.4, 55.4)
- added C4: 100n, Capacitor_SMD:C_0603_1608Metric_Pad1.08x0.95mm_HandSolder, F.Cu at (130.0, 89.9)
- added C6: 100n, Capacitor_SMD:C_0603_1608Metric_Pad1.08x0.95mm_HandSolder, F.Cu at (27.4, 55.4)
- added C7: 100n, Capacitor_SMD:C_0603_1608Metric_Pad1.08x0.95mm_HandSolder, F.Cu at (132.6, 35.1)
- added C8: 100n, Capacitor_SMD:C_0603_1608Metric_Pad1.08x0.95mm_HandSolder, F.Cu at (55.4, 73.2)
- added C9: 100n, Capacitor_SMD:C_0603_1608Metric_Pad1.08x0.95mm_HandSolder, F.Cu at (27.4, 89.9)
- added R14: 10k, Resistor_SMD:R_0603_1608Metric_Pad0.98x0.95mm_HandSolder, F.Cu at (126.5, 67.6)
- added R17: 10k, Resistor_SMD:R_0603_1608Metric_Pad0.98x0.95mm_HandSolder, F.Cu at (126.5, 65.0)
- added R18: 10k, Resistor_SMD:R_0603_1608Metric_Pad0.98x0.95mm_HandSolder, F.Cu at (126.5, 62.5)
- added R23: 10k, Resistor_SMD:R_0603_1608Metric_Pad0.98x0.95mm_HandSolder, F.Cu at (126.5, 59.9)
- added R24: 10k, Resistor_SMD:R_0603_1608Metric_Pad0.98x0.95mm_HandSolder, F.Cu at (126.5, 57.4)
- added R25: 10k, Resistor_SMD:R_0603_1608Metric_Pad0.98x0.95mm_HandSolder, F.Cu at (126.5, 54.9)
- added R26: 10k, Resistor_SMD:R_0603_1608Metric_Pad0.98x0.95mm_HandSolder, F.Cu at (126.5, 52.8)
- added R8: 10k, Resistor_SMD:R_0603_1608Metric_Pad0.98x0.95mm_HandSolder, F.Cu at (126.5, 70.1)
- C5: renamed from C05; footprint Capacitor_SMD:C_0201_0603Metric_Pad0.64x0.40mm_HandSolder -> Capacitor_SMD:C_0603_1608Metric_Pad1.08x0.95mm_HandSolder
- moved R20 114.5 mm to (137.2, 84.5)
- moved R13 113.8 mm to (160.3, 38.1), turned to 180 degrees
- moved C13 111.7 mm to (151.1, 46.4)
- moved C10 97.2 mm to (149.9, 29.2)
- moved R16 93.2 mm to (146.1, 46.4), turned to 180 degrees
- moved R22 93.2 mm to (136.5, 46.4), turned to 180 degrees
- moved R12 87.2 mm to (144.1, 29.8)
- moved R11 86.2 mm to (138.4, 29.8), turned to 180 degrees
- moved R19 81.5 mm to (102.6, 67.3), turned to 180 degrees
- moved R15 80.5 mm to (141.3, 46.4), turned to 180 degrees
- moved R10 76.4 mm to (126.4, 47.0)
- moved D1 74.2 mm to (65.4, 66.7), turned to 180 degrees
- moved R9 66.9 mm to (99.7, 57.1)
- moved R6 51.0 mm to (83.2, 54.0), turned to 180 degrees
- moved R5 50.9 mm to (69.8, 46.4)
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- renumbered IC01 to IC1, IC02 to IC2, IC03 to IC3, IC04 to IC4, IC05 to IC5, IC06 to IC6, IC07 to IC7, IC08 to IC8, IC09 to IC9, R01 to R1, R02 to R2, R03 to R3, R04 to R4, R05 to R5, R06 to R6, R07 to R7, R09 to R9
Connections:
- S2 pad 10: /~{DS0} -> /~{TRK00}
- S2 pad 12: /~{DS1} -> /~{WGATE}
- S2 pad 14: /~{DS2} -> /~{WDATA}
- S2 pad 16: /~{MTRON} -> /~{STEP}
- S2 pad 2: unconnected-(S2-Pad2) -> /~{RDY}
- S2 pad 20: /~{STEP} -> /~{MTRON}
- S2 pad 22: /~{WDATA} -> /~{DS2}
- S2 pad 24: /~{WGATE} -> /~{DS1}
- S2 pad 26: /~{TRK00} -> /~{DS0}
- S2 pad 28: /~{WPT} -> ~{INDEX}
- S2 pad 30: /~{RDATA} -> /~{DS3}
- S2 pad 32: /~{SIDE1} -> unconnected-(S2-Pad32)
- S2 pad 34: /~{RDY} -> unconnected-(S2-Pad34)
- S2 pad 4: unconnected-(S2-Pad4) -> /~{SIDE1}
- S2 pad 6: /~{DS3} -> /~{RDATA}
- S2 pad 8: ~{INDEX} -> /~{WPT}
Other:
- board text added: "8x10k"
