File: vortex-f1-d-clone.kicad_sch (KiCad schematic)
At the start: 39 parts, among them IC01 74LS136, IC02 74LS74, IC03 74LS85, IC04 27128, IC05 74LS14, IC06 74LS08, IC07 74LS25, IC08 74LS32, IC09 FDC_9229, IC10 uPD765AC, IC11 74LS01, IC12 74LS38, IC13 74LS07, IC14 74LS139

Commit message: Slightly rearrange to fit on smaller paper
Connections:
- net +5V: now also IC07.3
- net at IC02.11 (C), IC07.8: no longer IC07.3
- net ~{ROMOE}: now reaches IC04.22 (~{OE}), IC05.2
Other:
- title: (none) -> Vortex F1-D Reproduction
- moved on the sheet: C05, C10, C13, D1, IC01A, IC01B, IC01C, IC01D, IC01E, IC02A, IC02B, IC02C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

Commit message: PCB work
Parts:
- removed RN1: 10k, Resistor_THT:R_Array_SIP9, symbol Device:R_Network08
- added C1, C11, C12, C14, C15, C16, C17, C2, C3, C4, C6, C7, C8, C9: 100n, Capacitor_SMD:C_0603_1608Metric_Pad1.08x0.95mm_HandSolder, symbol Device:C_Small
- added R14, R17, R18, R23, R24, R25, R26, R8: 10k, Resistor_SMD:R_0603_1608Metric_Pad0.98x0.95mm_HandSolder, symbol Device:R_Small
- C10, C13: footprint (none) -> Capacitor_SMD:C_0805_2012Metric_Pad1.18x1.45mm_HandSolder
- C5: renamed from C05; footprint (none) -> Capacitor_SMD:C_0603_1608Metric_Pad1.08x0.95mm_HandSolder
- IC1: renamed from IC01; footprint (none) -> Package_DIP:DIP-14_W7.62mm_Socket
- IC10: footprint (none) -> Package_DIP:DIP-40_W15.24mm_Socket
- IC11, IC12, IC13: footprint (none) -> Package_DIP:DIP-14_W7.62mm_Socket
- IC14: footprint (none) -> Package_DIP:DIP-16_W7.62mm_Socket
- IC2: renamed from IC02; footprint (none) -> Package_DIP:DIP-14_W7.62mm_Socket
- IC3: renamed from IC03; footprint (none) -> Package_DIP:DIP-16_W7.62mm_Socket
- IC5: renamed from IC05; footprint (none) -> Package_DIP:DIP-14_W7.62mm_Socket
- IC6: renamed from IC06; footprint (none) -> Package_DIP:DIP-14_W7.62mm_Socket
- IC7: renamed from IC07; footprint (none) -> Package_DIP:DIP-14_W7.62mm_Socket
- IC8: renamed from IC08; footprint (none) -> Package_DIP:DIP-14_W7.62mm_Socket
- IC9: renamed from IC09; footprint (none) -> Package_DIP:DIP-20_W7.62mm_Socket
- R1: renamed from R01; footprint (none) -> Resistor_SMD:R_0603_1608Metric_Pad0.98x0.95mm_HandSolder
- R10, R11, R12, R13, R15, R16, R19, R20, R21, R22: footprint (none) -> Resistor_SMD:R_0603_1608Metric_Pad0.98x0.95mm_HandSolder
- R2: renamed from R02; footprint (none) -> Resistor_SMD:R_0603_1608Metric_Pad0.98x0.95mm_HandSolder
- R3: renamed from R03; footprint (none) -> Resistor_SMD:R_0603_1608Metric_Pad0.98x0.95mm_HandSolder
- R4: renamed from R04; footprint (none) -> Resistor_SMD:R_0603_1608Metric_Pad0.98x0.95mm_HandSolder
- R5: renamed from R05; footprint (none) -> Resistor_SMD:R_0603_1608Metric_Pad0.98x0.95mm_HandSolder
- R6: renamed from R06; footprint (none) -> Resistor_SMD:R_0603_1608Metric_Pad0.98x0.95mm_HandSolder
- R7: renamed from R07; footprint (none) -> Resistor_SMD:R_0603_1608Metric_Pad0.98x0.95mm_HandSolder
- R9: renamed from R09; footprint (none) -> Resistor_SMD:R_0603_1608Metric_Pad0.98x0.95mm_HandSolder
- S1: footprint (none) -> Connector_PinHeader_2.54mm:PinHeader_2x25_P2.54mm_Vertical
- S2: footprint (none) -> Connector_IDC:IDC-Header_2x17_P2.54mm_Vertical
- renumbered IC04 to IC4
Connections:
- net +5V: now also C1.1, C11.1, C12.1, C14.1, C15.1, C16.1, C17.1, C2.1, C3.1, C4.1, C6.1, C7.1, C8.1, C9.1, R14.2, R17.2, R18.2, R23.2, R24.2, R25.2, R26.2, R8.2
- net D0: now also R8.1
- net D1: now also R14.1
- net D2: now also R17.1
- net D3: now also R18.1
- net D4: now also R23.1
- net D5: now also R24.1
- net D6: now also R25.1
- net D7: now also R26.1
- net GND: now also C1.2, C11.2, C12.2, C14.2, C15.2, C16.2, C17.2, C2.2, C3.2, C4.2, C6.2, C7.2, C8.2, C9.2
- net ~{DS0}: now also S2.26 (Pin_26); no longer S2.10 (Pin_10)
- net ~{DS1}: now also S2.24 (Pin_24); no longer S2.12 (Pin_12)
- net ~{DS2}: now also S2.22 (Pin_22); no longer S2.14 (Pin_14)
- net ~{DS3}: now also S2.30 (Pin_30); no longer S2.6 (Pin_6)
- net ~{INDEX}: now also S2.28 (Pin_28); no longer S2.8 (Pin_8)
- net ~{MTRON}: now also S2.20 (Pin_20); no longer S2.16 (Pin_16)
- net ~{RDATA}: now also S2.6 (Pin_6); no longer S2.30 (Pin_30)
- net ~{RDY}: now also S2.2 (Pin_2); no longer S2.34 (Pin_34)
- net ~{SIDE1}: now also S2.4 (Pin_4); no longer S2.32 (Pin_32)
- net ~{STEP}: now also S2.16 (Pin_16); no longer S2.20 (Pin_20)
- net ~{TRK00}: now also S2.10 (Pin_10); no longer S2.26 (Pin_26)
- net ~{WDATA}: now also S2.14 (Pin_14); no longer S2.22 (Pin_22)
- net ~{WGATE}: now also S2.12 (Pin_12); no longer S2.24 (Pin_24)
- net ~{WPT}: now also S2.8 (Pin_8); no longer S2.28 (Pin_28)
Other:
- moved on the sheet: S2
