File: vortex-f1-d-no-rom.kicad_pcb (KiCad board)
At the start: 2 copper layers, 111.9 x 64.1 mm, 47 parts, among them IC1 74LS136, IC10 uPD765AC, IC11 74HCT688, IC12 74LS38, IC13 74LS07, IC14 74LS139, IC15 74HCT688, IC2 74LS74, IC5 74LS14, IC6 74LS08, IC7 74HCT688, IC8 74LS32, IC9 FDC_9229, X1 8Mhz

Commit message: Silkscreen work
Parts:
- IC10: value uPD765AC -> μPD765AC
- IC9: value FDC_9229 -> FDC 9229
Other:
- board text added: "8x10k"
- board text added: "CPC-FDC v0.1"
- board text added: "https://github.com/hanshuebner/vortex-f1-d-clone"
