File: vortex-f1-d-no-rom.kicad_pcb (KiCad board)
At the start: 2 copper layers, 111.9 x 64.1 mm, 47 parts, among them IC1 74LS136, IC10 μPD765AC, IC11 74HCT688, IC12 74LS38, IC13 74LS07, IC14 74LS139, IC15 74HCT688, IC2 74LS74, IC5 74LS14, IC6 74LS08, IC7 74HCT688, IC8 74LS32, IC9 FDC 9229, X1 8Mhz

Commit message: sent TTL variant to aisler for production
Parts:
- IC10: value μPD765AC -> uPD765AC
- IC9: value FDC 9229 -> FDC_9229
- renumbered C12 to C10, C14 to C11, C15 to C12, C16 to C13, C6 to C5, C7 to C6, C8 to C7, C9 to C8, C11 to C9
Connections:
- net ~{MOTOR} renamed MOTOR
- IC10 pad 35: READY -> RDY
- IC2 pad 3: ~{MOTCS} -> Net-(IC2-Pad3)
- IC5 pad 1: (no net) -> ~{MOTCS}
- IC5 pad 2: (no net) -> Net-(IC2-Pad3)
- IC5 pad 8: READY -> RDY
- IC6 pad 9: READY -> RDY
- S1 pad 39: READY -> /READY
Routing:
- net READY: track 91.5 -> 0.00 mm, vias 4 -> 0
- net RDY: track 0.00 -> 63.0 mm, vias 0 -> 3
- net Net-(IC2-Pad3): track 0.00 -> 55.1 mm, vias 0 -> 3
- net ~{MOTCS}: track 6.39 -> 49.9 mm, vias 0 -> 3
- net GND: track 129.6 -> 156.3 mm, vias 54 -> 69
- net SIDE: track 46.6 -> 49.3 mm
- net ~{TRK00}: track 77.5 -> 79.5 mm
- net WE: track 40.9 -> 38.9 mm, vias 2 -> 3
- net /D6: track 55.4 -> 53.7 mm
- net Net-(IC13-Pad11): track 66.9 -> 68.5 mm
- net Net-(IC13-Pad5): track 73.6 -> 74.7 mm
- net Net-(IC13-Pad9): track 66.5 -> 67.5 mm
- net Net-(IC5-Pad10): track 47.7 -> 48.7 mm
- net MOTOR: track 98.0 -> 98.9 mm
- net INDEX: track 52.7 -> 51.9 mm
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
Commit message: Update version number
Other:
- board text added: "CPC-FDC v0.2"
- board text removed: "CPC-FDC v0.1"
Changed lines of the file:
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@@
     (effects (font (size 1.5 1) (thickness 0.15)) (justify mirror))
   )
-  (gr_text "CPC-FDC v0.1" (at 104.648 71.12) (layer "F.SilkS")
+  (gr_text "CPC-FDC v0.2" (at 104.648 71.12) (layer "F.SilkS")
     (effects (font (size 3 2) (thickness 0.3)))
   )
