File: vortex-f1-d-cpld.kicad_sch (KiCad schematic)
At the start: 50 parts, among them J1 JTAG, J2 CONFIG, U1 FDC 9229, U2 XC9572XL, U3 AZ1117-3.3, U4 uPD765AC, U5 74LS06N, U6 74LS06N, U7 SN74LS07N, X1 8Mhz

Commit message: Version with ROM
Parts:
- removed J1: JTAG, Connector_PinHeader_2.00mm:PinHeader_2x07_P2.00mm_Vertical, symbol Connector_Generic:Conn_02x07_Odd_Even
- removed J2: CONFIG, Connector_PinHeader_2.54mm:PinHeader_2x04_P2.54mm_Vertical, symbol Connector_Generic:Conn_02x04_Odd_Even
- removed LED2: LED2, LED_SMD:LED_0805_2012Metric_Pad1.15x1.40mm_HandSolder, symbol Device:LED_Small_Filled
- removed LED3: LED3, LED_SMD:LED_0805_2012Metric_Pad1.15x1.40mm_HandSolder, symbol Device:LED_Small_Filled
- removed LED4: LED4, LED_SMD:LED_0805_2012Metric_Pad1.15x1.40mm_HandSolder, symbol Device:LED_Small_Filled
- removed R2, R3, R4: 180, Resistor_SMD:R_0603_1608Metric_Pad0.98x0.95mm_HandSolder, symbol Device:R_Small
- added C12: 100n, Capacitor_SMD:C_0603_1608Metric_Pad1.08x0.95mm_HandSolder, symbol Device:C_Small
- added J1: JTAG, Connector_PinHeader_2.54mm:PinHeader_2x03_P2.54mm_Vertical, symbol Connector_Generic:Conn_02x03_Counter_Clockwise
- added JP1: ~{VORTEX}/CPC, Jumper:SolderJumper-2_P1.3mm_Open_RoundedPad1.0x1.5mm, symbol Jumper:SolderJumper_2_Open
- added U5: AM29F010, Package_LCC:PLCC-32_THT-Socket, symbol Memory_Flash:29F010-TSOP-SP
- LED1: value LED1 -> STATUS
- U6: renamed from U5; footprint Package_SO:SOIC-14_3.9x8.7mm_P1.27mm -> Package_SO:SSOP-14_5.3x6.2mm_P0.65mm
- U7: footprint Package_SO:SOIC-14_3.9x8.7mm_P1.27mm -> Package_SO:SSOP-14_5.3x6.2mm_P0.65mm
- U8: renamed from U6; footprint Package_SO:SOIC-14_3.9x8.7mm_P1.27mm -> Package_SO:SSOP-14_5.3x6.2mm_P0.65mm
- renumbered R13 to R10, R14 to R11, R15 to R12, R16 to R13, R17 to R14, R18 to R15, R19 to R16, R20 to R17, R21 to R18, R22 to R19, R5 to R2, R23 to R20, R6 to R3, R7 to R4, R8 to R5, R9 to R6, R10 to R7, R11 to R8, R12 to R9
Connections:
- net +3.3V: now also J1.1 (Pin_1)
- net +5V: now also C12.1, U5.32 (VCC)
- net A0: now also U5.12 (A0)
- net A1: now also U5.11 (A1)
- net A10: now also U5.23 (A10)
- net A11: now also U5.25 (A11)
- net A12: now also U5.4 (A12)
- net A13: now also U5.28 (A13)
- net A2: now also U5.10 (A2)
- net A3: now also U5.9 (A3)
- net A4: now also U5.8 (A4)
- net A5: now also U5.7 (A5)
- net A6: now also U5.6 (A6)
- net A7: now also U5.5 (A7)
- net A8: now also U5.27 (A8)
- net A9: now also U5.26 (A9)
- net CLK4: no longer U2.16 (I/O/GCK2)
- net D0: now also U5.13 (D0)
- net D1: now also U5.14 (D1)
- net D2: now also U5.15 (D2)
- net D3: now also U5.17 (D3)
- net D4: now also U5.18 (D4)
- net D5: now also U5.19 (D5)
- net D6: now also U5.20 (D6)
- net D7: now also U5.21 (D7)
- net GND: now also C12.2, J1.3 (Pin_3), JP1.1 (A), U5.16 (GND)
- net LED1: now also U2.16 (I/O/GCK2); no longer U2.22 (P22)
- net READY: no longer U4.35 (READY), U6.2
- net TCK: now also J1.5 (Pin_5)
- net TDI: now also J1.2 (Pin_2)
- net TDO: now also J1.4 (Pin_4)
- net TMS: now also J1.6 (Pin_6)
- net ROMA16: now reaches U2.27 (P27)
- net ROMA16: now also U5.2 (A16)
- net ROMA15: now reaches U2.31 (P31)
- net ROMA15: now also U5.3 (A15)
- net ROMA14: now reaches U2.32 (P32)
- net ROMA14: now also U5.29 (A14)
- net CFG1 renamed ~{VORTEX}/CPC
- net ~{VORTEX}/CPC: now also JP1.2 (B)
- net CFG2: no longer names the net of U2.19 (P19)
- net CFG3: no longer names the net of U2.18 (P18)
- net CFG4: no longer names the net of U2.17 (I/O/GCK3)
- net LED3 renamed ~{ROMOE}
- net ~{ROMOE}: now also U5.24 (OE)
- net LED4 renamed ~{ROMCE}
- net ~{ROMCE}: now also U5.22 (CE)
- new net RDY: U4.35 (READY), U6.2
- new net ~{ROMWE}: U2.22 (P22), U5.31 (WE)
- no-connect marks 13 -> 10

Commit message: Layout with ROM redone
Parts:
- added D1: 1N4148W, Diode_SMD:D_SOD-123, symbol Diode:1N4148W
Connections:
- net LED2 is gone; now on net TRK00: U2.23 (P23)
- net A0: now also U2.33 (P33); no longer U2.50 (P50)
- net A1: now also U2.34 (P34); no longer U2.49 (P49)
- net A10: now also U2.43 (P43); no longer U2.39 (P39)
- net A11: no longer U2.38 (P38)
- net A12: no longer U2.36 (P36)
- net A13: now also U2.44 (P44); no longer U2.35 (P35)
- net A14: no longer U2.34 (P34)
- net A15: now also U2.45 (P45); no longer U2.33 (P33)
- net A2: now also U2.35 (P35); no longer U2.48 (P48)
- net A3: now also U2.36 (P36); no longer U2.47 (P47)
- net A4: now also U2.38 (P38); no longer U2.46 (P46)
- net A5: now also U2.39 (P39); no longer U2.45 (P45)
- net A6: now also U2.40 (P40); no longer U2.44 (P44)
- net A7: now also U2.42 (P42); no longer U2.43 (P43)
- net A8: now also U2.18 (P18); no longer U2.42 (P42)
- net A9: now also U2.17 (I/O/GCK3); no longer U2.40 (P40)
- net CLK4: now also U2.58 (P58)
- net D0: now also U2.46 (P46); no longer U2.51 (P51)
- net FLTR/STEP: now also U2.2 (I/O/GTS2); no longer U2.59 (P59)
- net FLT/TRK0: now also U2.4 (P4); no longer U2.2 (I/O/GTS2)
- net LED1: now also U2.15 (I/O/GCK1); no longer U2.16 (I/O/GCK2)
- net MTRON: now also U2.24 (P24); no longer U2.7 (P7)
- net READY: now also U2.51 (P51); no longer U2.1 (P1)
- net RESET: now also U2.8 (P8); no longer U2.62 (P62)
- net ROMA14: now also U2.59 (P59); no longer U2.32 (P32)
- net ROMA15: now also U2.64 (I/O/GSR); no longer U2.31 (P31)
- net ROMA16: now also U2.63 (P63); no longer U2.27 (P27)
- net ROMDIS: now also D1.1 (K)
- net STEP: now also U2.20 (P20), U6.9; no longer U2.12 (P12), U6.13
- net TRK00: now also U6.12; no longer U2.15 (I/O/GCK1), U6.8
- net US0: now also U2.6 (P6); no longer U2.4 (P4)
- net WE: now also U2.7 (P7); no longer U2.64 (I/O/GSR)
- net WGATE: now also U2.22 (P22); no longer U2.13 (P13)
- net ~{DS0'}: now also U2.31 (P31); no longer U2.8 (P8)
- net ~{DS1'}: now also U2.27 (P27), U7.13; no longer U2.9 (P9), U7.9
- net ~{DS1}: now also U7.12; no longer U7.8
- net ~{DS2'}: now also U2.25 (P25); no longer U2.10 (P10)
- net ~{DS3'}: now also U2.32 (P32), U7.9; no longer U2.11 (P11), U7.13
- net ~{DS3}: now also U7.8; no longer U7.12
- net ~{FDCCS}: now also U2.11 (P11); no longer U2.63 (P63)
- net ~{IORD}: now also U2.9 (P9); no longer U2.60 (P60)
- net ~{IORQ}: now also U2.48 (P48); no longer U2.52 (P52)
- net ~{IOWR}: now also U2.10 (P10); no longer U2.61 (P61)
- net ~{MREQ}: now also U2.47 (P47)
- net ~{RD}: now also U2.49 (P49); no longer U2.57 (P57)
- net ~{ROMCE}: now also U2.62 (P62); no longer U2.25 (P25)
- net ~{ROMEN}: now also U2.52 (P52)
- net ~{ROMOE}: now also U2.61 (P61); no longer U2.24 (P24)
- net ~{ROMWE}: now also U2.60 (P60); no longer U2.22 (P22)
- net ~{RSET}: now also U2.56 (P56); no longer U2.58 (P58)
- net ~{RW}/SEEK: now also U2.1 (P1); no longer U2.6 (P6)
- net ~{STEP}: now also U6.8; no longer U6.12
- net ~{TRK00}: now also U6.13; no longer U6.9
- net ~{VORTEX}/CPC: now also U2.16 (I/O/GCK2); no longer U2.20 (P20)
- net ~{WR}: now also U2.50 (P50); no longer U2.56 (P56)
- new net: D1.2 (A), U2.57 (P57)
Other:
- moved on the sheet: U2
