File: vortex-f1-d-no-rom.kicad_sch (KiCad schematic)
At the start: 60 parts, among them IC1 74LS136, IC10 uPD765AC, IC11 74LS01, IC12 74LS38, IC13 74LS07, IC14 74LS139, IC2 74LS74, IC3 74LS85, IC4 27128, IC5 74LS14, IC6 74LS08, IC7 74LS25, IC8 74LS32, IC9 FDC_9229

Commit message: ROMless variant schematic, CPC Dandanator CPLD
Parts:
- removed C10: 47u 16V, Capacitor_SMD:C_0805_2012Metric_Pad1.18x1.45mm_HandSolder, symbol Device:C_Polarized_Small
- removed C13: 4.7u 25V, Capacitor_SMD:C_0805_2012Metric_Pad1.18x1.45mm_HandSolder, symbol Device:C_Polarized_Small
- removed C5: 47p, Capacitor_SMD:C_0603_1608Metric_Pad1.08x0.95mm_HandSolder, symbol Device:C_Small
- removed D1: 1N4148, Diode_THT:D_DO-35_SOD27_P7.62mm_Horizontal, symbol Diode:1N4148
- removed unit 2 of IC1
- removed unit 3 of IC11
- removed unit 1 of IC11
- removed unit 4 of IC11
- removed unit 2 of IC11
- removed unit 1 of IC14
- removed unit 1 of IC2
- removed unit 2 of IC2
- removed IC3: 74LS85, Package_DIP:DIP-16_W7.62mm_Socket, symbol 74xx:74LS85
- removed IC4: 27128, Package_DIP:DIP-28_W15.24mm, symbol Memory_EPROM:27128
- removed unit 2 of IC5
- removed unit 1 of IC5
- removed unit 1 of IC6
- removed unit 1 of IC7
- removed unit 2 of IC7
- removed unit 3 of IC8
- removed unit 2 of IC8
- removed R11, R15, R21, R22: 1k, Resistor_SMD:R_0603_1608Metric_Pad0.98x0.95mm_HandSolder, symbol Device:R_Small
- removed R12, R16, R2, R3, R4, R5: 680, Resistor_SMD:R_0603_1608Metric_Pad0.98x0.95mm_HandSolder, symbol Device:R_Small
- added R? (x2): 680, Resistor_SMD:R_0603_1608Metric_Pad0.98x0.95mm_HandSolder, symbol Device:R_Small
- added U?: XC95144XL-TQ100, Package_QFP:TQFP-100_14x14mm_P0.5mm, symbol CPLD_Xilinx:XC95144XL-TQ100
- added X?: 8Mhz, Oscillator:Oscillator_SMD_EuroQuartz_XO91-4Pin_7.0x5.0mm, symbol Oscillator:XO91
Connections:
- net +5V: now also IC1.12, IC1.9, R?.2, R?.2; no longer IC1.10, IC1.13
- net READY: now also IC6.9; no longer IC6.10
- net ~{INDEX}: now also R?.1
- net ~{WPT}: now also R?.1
- net at IC6.8: now also IC1.13; no longer IC1.12
- net WE: now reaches IC10.25 (WE)
- net WE: now also IC6.10; no longer IC6.9
- net ~{CLKIN}: now reaches IC9.11 (~{CLKIN})
- net ~{CLKIN}: now also X?.3 (OUT)
- net ~{IOWR}: now reaches IC10.3 (~{WR}), IC8.11
- net at IC6.11: now also IC1.10; no longer IC1.9
- net FLTR/STEP: now reaches IC10.37 (FLTR/STEP), IC6.12
- net ~{RW}/SEEK: now reaches IC10.39 (~{RW}/SEEK), IC6.13
- net ~{RW}/SEEK: now also IC6.5; no longer IC6.4
- net ~{MOTOR}: now reaches IC1.2
- net DSKD: now reaches IC13.2, IC9.1 (DSKD), R9.1
- net LCT/DIR: now reaches IC10.38 (LCT/DIR), IC12.1, IC12.2
- net ~{IORD}: now reaches IC10.2 (~{RD}), IC8.3
- net MFM: now reaches IC10.26 (MFM), IC9.4 (DENS)
- net WDOUT: now reaches IC12.12, IC12.13, IC9.7 (WDOUT)
- net SIDE: now reaches IC10.27 (SIDE), IC12.4, IC12.5
- net RESET: now reaches IC10.1 (RESET), IC10.16 (TC), IC5.6
- net WPRT/2SIDE: now reaches IC10.34 (WPRT/2SIDE), IC12.8, R19.1
- net ~{CS}: now reaches IC10.4 (~{CS})
- net US0: now reaches IC10.28 (US0), IC14.13 (A1)
- net US1: now reaches IC10.29 (US1), IC14.14 (A0)
- net FLT/TRK0: now reaches IC10.33 (FLT/TRK0), IC6.6
- net TRK00: no longer names the net of IC5.10
- net TRK00: now also IC6.4; no longer IC6.5
- no-connect marks 17 -> 9
Other:
- note added: "I/O Port Usage: &FBF6 Status &FBF7 Data &FA7E Motor"
- moved on the sheet: IC10, IC12A, IC12B, IC12C, IC12D, IC13A, IC13B, IC13C, IC13D, IC13E, IC14B, IC1A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

Commit message: routed no-rom board
Parts:
- removed C17: 100n, Capacitor_SMD:C_0603_1608Metric_Pad1.08x0.95mm_HandSolder, symbol Device:C_Small
- removed IC11: 74LS01, Package_DIP:DIP-14_W7.62mm_Socket, symbol 74xx:74LS01
- removed unit 6 of IC13
- removed IC7: 74LS25, Package_DIP:DIP-14_W7.62mm_Socket, symbol 74xx:74LS25
- removed U?: XC95144XL-TQ100, Package_QFP:TQFP-100_14x14mm_P0.5mm, symbol CPLD_Xilinx:XC95144XL-TQ100
- added IC11, IC15, IC7: 74HCT688, Package_DIP:DIP-20_W7.62mm_Socket, symbol 74xx:74HCT688
- added unit 1 of IC2
- gave numbers to parts that had none: 3
- renumbered C12 to C10, C14 to C11, C15 to C12, C16 to C13, C6 to C5, C7 to C6, C8 to C7, C9 to C8, C11 to C9
Connections:
- net +5V: now also X1.1 (EN), X1.4 (V+), IC11.11 (P4), IC11.13 (P5), IC11.15 (P6), IC11.20 (VCC), IC11.6 (P2), IC11.8 (P3), IC15.13 (P5), IC15.15 (P6), IC15.2 (P0), IC15.20 (VCC), IC15.4 (P1), IC15.6 (P2), IC15.8 (P3), IC2.4 (~{S}), IC7.11 (P4), IC7.15 (P6), IC7.17 (P7), IC7.2 (P0), IC7.20 (VCC), IC7.4 (P1), IC7.6 (P2), IC7.8 (P3)
- net A0: now also IC11.18 (R7)
- net A1: now also IC11.16 (R6), IC15.16 (R6)
- net A10: now also IC7.14 (R5)
- net A11: now also IC7.12 (R4)
- net A12: now also IC7.9 (R3)
- net A13: now also IC7.7 (R2)
- net A14: now also IC7.5 (R1)
- net A15: now also IC7.3 (R0)
- net A2: now also IC11.14 (R5), IC15.14 (R5)
- net A3: now also IC11.12 (R4), IC15.12 (R4)
- net A4: now also IC11.9 (R3), IC15.9 (R3)
- net A5: now also IC11.7 (R2), IC15.7 (R2)
- net A6: now also IC7.18 (R7)
- net A7: now also IC11.5 (R1), IC15.5 (R1)
- net A8: now also IC11.3 (R0), IC15.3 (R0)
- net A9: now also IC7.16 (R6)
- net D0: now also IC2.2 (D)
- net GND: now also X1.2 (GND), IC11.10 (GND), IC11.17 (P7), IC11.2 (P0), IC11.4 (P1), IC15.10 (GND), IC15.11 (P4), IC15.17 (P7), IC15.18 (R7), IC7.1 (G), IC7.10 (GND), IC7.13 (P5)
- net ~{MOTOR}: now also IC2.5 (Q)
- net ~{RSET}: now also IC2.1 (~{R})
- net ~{CS} renamed ~{FDCCS}
- net ~{FDCCS}: now also IC15.19 (P=R)
- new net: IC11.1 (G), IC15.1 (G), IC7.19 (P=R)
- new net ~{MOTCS}: IC11.19 (P=R), IC2.3 (C)
- no-connect marks 9 -> 8
Other:
- moved on the sheet: IC12E, IC13G, IC14C, IC8E

Commit message: sent TTL variant to aisler for production
Parts:
- added unit 1 of IC5
Connections:
- net READY: no longer IC10.35 (READY), IC5.8, IC6.9
- net ~{MOTCS}: now also IC5.1; no longer IC2.3 (C)
- net ~{MOTOR} renamed MOTOR
- new net: IC2.3 (C), IC5.2
- new net RDY: IC10.35 (READY), IC5.8, IC6.9
Other:
- moved on the sheet: IC2A
Changed lines of the file:
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@@
   (no_connect (at 261.62 104.14))
   (no_connect (at 261.62 109.22))
-  (no_connect (at 76.2 100.33))
+  (no_connect (at 97.79 108.585))
   (no_connect (at 287.02 95.25))
   (no_connect (at 287.02 123.19))
@@
     (stroke (width 0) (type default) (color 0 0 0 0))
   )
+  (wire (pts (xy 90.17 118.745) (xy 90.17 113.665))
+    (stroke (width 0) (type default) (color 0 0 0 0))
+  )
   (wire (pts (xy 162.56 152.4) (xy 153.67 152.4))
     (stroke (width 0) (type default) (color 0 0 0 0))
@@
     (stroke (width 0) (type default) (color 0 0 0 0))
   )
+  (wire (pts (xy 49.53 106.045) (xy 55.245 106.045))
+    (stroke (width 0) (type default) (color 0 0 0 0))
+  )
   (wire (pts (xy 356.87 311.15) (xy 356.87 313.69))
     (stroke (width 0) (type default) (color 0 0 0 0))
@@
     (stroke (width 0) (type default) (color 0 0 0 0))
   )
-  (wire (pts (xy 68.58 110.49) (xy 68.58 105.41))
-    (stroke (width 0) (type default) (color 0 0 0 0))
-  )
   (wire (pts (xy 548.64 62.23) (xy 552.45 62.23))
     (stroke (width 0) (type default) (color 0 0 0 0))
@@
     (stroke (width 0) (type default) (color 0 0 0 0))
   )
-  (wire (pts (xy 68.58 86.36) (xy 68.58 90.17))
+  (wire (pts (xy 90.17 94.615) (xy 90.17 98.425))
     (stroke (width 0) (type default) (color 0 0 0 0))
   )
@@
     (stroke (width 0) (type default) (color 0 0 0 0))
   )
-  (wire (pts (xy 62.23 110.49) (xy 68.58 110.49))
-    (stroke (width 0) (type default) (color 0 0 0 0))
-  )
   (wire (pts (xy 91.44 67.31) (xy 91.44 69.85))
     (stroke (width 0) (type default) (color 0 0 0 0))
@@
     (stroke (width 0) (type default) (color 0 0 0 0))
   )
-  (wire (pts (xy 58.42 97.79) (xy 60.96 97.79))
+  (wire (pts (xy 70.485 106.045) (xy 82.55 106.045))
     (stroke (width 0) (type default) (color 0 0 0 0))
   )
@@
     (stroke (width 0) (type default) (color 0 0 0 0))
   )
-  (wire (pts (xy 58.42 95.25) (xy 60.96 95.25))
+  (wire (pts (xy 80.01 103.505) (xy 82.55 103.505))
     (stroke (width 0) (type default) (color 0 0 0 0))
   )
@@
     (stroke (width 0) (type default) (color 0 0 0 0))
   )
-  (wire (pts (xy 76.2 95.25) (xy 80.01 95.25))
+  (wire (pts (xy 97.79 103.505) (xy 101.6 103.505))
     (stroke (width 0) (type default) (color 0 0 0 0))
   )
@@
     (stroke (width 0) (type default) (color 0 0 0 0))
   )
+  (wire (pts (xy 80.01 118.745) (xy 90.17 118.745))
+    (stroke (width 0) (type default) (color 0 0 0 0))
+  )
   (wire (pts (xy 552.45 49.53) (xy 552.45 52.07))
     (stroke (width 0) (type default) (color 0 0 0 0))
@@
   )
   (text "I/O Port Usage:\n\n&FBF6 Status\n&FBF7 Data\n&FA7E Motor"
-    (at 106.68 125.73 0)
+    (at 107.95 90.17 0)
     (effects (font (size 2.54 2.54)) (justify left bottom))
   )
@@
     )
   )
-  (global_label "READY" (shape input) (at 292.1 100.33 0) (fields_autoplaced)
+  (global_label "RDY" (shape input) (at 292.1 100.33 0) (fields_autoplaced)
     (effects (font (size 1.27 1.27)) (justify left))
-    (property "Intersheet References" "${INTERSHEET_REFS}" (id 0) (at 300.3793 100.2506 0)
+    (property "Intersheet References" "${INTERSHEET_REFS}" (id 0) (at 298.1417 100.2506 0)
       (effects (font (size 1.27 1.27)) (justify left) hide)
     )
@@
     )
   )
-  (global_label "D0" (shape input) (at 58.42 95.25 180) (fields_autoplaced)
+  (global_label "D0" (shape input) (at 80.01 103.505 180) (fields_autoplaced)
     (effects (font (size 1.27 1.27)) (justify right))
-    (property "Intersheet References" "${INTERSHEET_REFS}" (id 0) (at 53.5274 95.1706 0)
+    (property "Intersheet References" "${INTERSHEET_REFS}" (id 0) (at 75.1174 103.4256 0)
       (effects (font (size 1.27 1.27)) (justify right) hide)
     )
@@
     )
   )
-  (global_label "~{MOTCS}" (shape input) (at 58.42 97.79 180) (fields_autoplaced)
+  (global_label "~{MOTCS}" (shape input) (at 49.53 106.045 180) (fields_autoplaced)
     (effects (font (size 1.27 1.27)) (justify right))
-    (property "Intersheet References" "${INTERSHEET_REFS}" (id 0) (at 49.7779 97.7106 0)
+    (property "Intersheet References" "${INTERSHEET_REFS}" (id 0) (at 40.8879 105.9656 0)
       (effects (font (size 1.27 1.27)) (justify right) hide)
     )
@@
     )
   )
-  (global_label "~{MOTOR}" (shape output) (at 80.01 95.25 0) (fields_autoplaced)
+  (global_label "MOTOR" (shape output) (at 101.6 103.505 0) (fields_autoplaced)
     (effects (font (size 1.27 1.27)) (justify left))
-    (property "Intersheet References" "${INTERSHEET_REFS}" (id 0) (at 88.7731 95.1706 0)
+    (property "Intersheet References" "${INTERSHEET_REFS}" (id 0) (at 110.3631 103.4256 0)
       (effects (font (size 1.27 1.27)) (justify left) hide)
     )
@@
     )
   )
-  (global_label "~{MOTOR}" (shape input) (at 372.11 119.38 180) (fields_autoplaced)
+  (global_label "MOTOR" (shape input) (at 372.11 119.38 180) (fields_autoplaced)
     (effects (font (size 1.27 1.27)) (justify right))
     (property "Intersheet References" "${INTERSHEET_REFS}" (id 0) (at 363.3469 119.3006 0)
@@
     )
   )
-  (global_label "READY" (shape output) (at 350.52 171.45 180) (fields_autoplaced)
+  (global_label "RDY" (shape output) (at 350.52 171.45 180) (fields_autoplaced)
     (effects (font (size 1.27 1.27)) (justify right))
-    (property "Intersheet References" "${INTERSHEET_REFS}" (id 0) (at 342.2407 171.5294 0)
+    (property "Intersheet References" "${INTERSHEET_REFS}" (id 0) (at 344.4783 171.3706 0)
       (effects (font (size 1.27 1.27)) (justify right) hide)
     )
@@
     )
   )
-  (global_label "~{RSET}" (shape input) (at 62.23 110.49 180) (fields_autoplaced)
+  (global_label "~{RSET}" (shape input) (at 80.01 118.745 180) (fields_autoplaced)
     (effects (font (size 1.27 1.27)) (justify right))
-    (property "Intersheet References" "${INTERSHEET_REFS}" (id 0) (at 55.2207 110.4106 0)
+    (property "Intersheet References" "${INTERSHEET_REFS}" (id 0) (at 73.0007 118.6656 0)
       (effects (font (size 1.27 1.27)) (justify right) hide)
     )
@@
     (pin "1")
   )
-  (symbol (lib_id "74xx:74LS74") (at 68.58 97.79 0) (unit 1)
+  (symbol (lib_id "74xx:74LS74") (at 90.17 106.045 0) (unit 1)
     (in_bom yes) (on_board yes) (fields_autoplaced)
-    (property "Reference" "IC2" (id 0) (at 70.5994 87.63 0)
+    (property "Reference" "IC2" (id 0) (at 92.1894 95.885 0)
       (effects (font (size 1.27 1.27)) (justify left))
     )
-    (property "Value" "74LS74" (id 1) (at 70.5994 90.17 0)
+    (property "Value" "74LS74" (id 1) (at 92.1894 98.425 0)
       (effects (font (size 1.27 1.27)) (justify left))
     )
-    (property "Footprint" "Package_DIP:DIP-14_W7.62mm_Socket" (id 2) (at 68.58 97.79 0)
+    (property "Footprint" "Package_DIP:DIP-14_W7.62mm_Socket" (id 2) (at 90.17 106.045 0)
       (effects (font (size 1.27 1.27)) hide)
     )
-    (property "Datasheet" "74xx/74hc_hct74.pdf" (id 3) (at 68.58 97.79 0)
+    (property "Datasheet" "74xx/74hc_hct74.pdf" (id 3) (at 90.17 106.045 0)
       (effects (font (size 1.27 1.27)) hide)
     )
@@
     (pin "9")
   )
+  (symbol (lib_id "74xx:74LS14") (at 62.865 106.045 0) (unit 1)
+    (in_bom yes) (on_board yes) (fields_autoplaced)
+    (property "Reference" "IC5" (id 0) (at 62.865 97.155 0))
+    (property "Value" "74LS14" (id 1) (at 62.865 99.695 0))
+    (property "Footprint" "Package_DIP:DIP-14_W7.62mm_Socket" (id 2) (at 62.865 106.045 0)
+      (effects (font (size 1.27 1.27)) hide)
+    )
+    (property "Datasheet" "http://www.ti.com/lit/gpn/sn74LS14" (id 3) (at 62.865 106.045 0)
+      (effects (font (size 1.27 1.27)) hide)
+    )
+    (pin "1")
+    (pin "2")
+    (pin "3")
+    (pin "4")
+    (pin "5")
+    (pin "6")
+    (pin "8")
+    (pin "9")
+    (pin "10")
+    (pin "11")
+    (pin "12")
+    (pin "13")
+    (pin "14")
+    (pin "7")
+  )
   (symbol (lib_id "power:+5V") (at 182.88 72.39 0) (unit 1)
     (in_bom yes) (on_board yes) (fields_autoplaced)
@@
     (pin "7")
   )
-  (symbol (lib_id "power:+5V") (at 68.58 86.36 0) (unit 1)
+  (symbol (lib_id "power:+5V") (at 90.17 94.615 0) (unit 1)
     (in_bom yes) (on_board yes) (fields_autoplaced)
-    (property "Reference" "#PWR01" (id 0) (at 68.58 90.17 0)
+    (property "Reference" "#PWR01" (id 0) (at 90.17 98.425 0)
       (effects (font (size 1.27 1.27)) hide)
     )
-    (property "Value" "+5V" (id 1) (at 68.58 81.28 0))
-    (property "Footprint" "" (id 2) (at 68.58 86.36 0)
+    (property "Value" "+5V" (id 1) (at 90.17 89.535 0))
+    (property "Footprint" "" (id 2) (at 90.17 94.615 0)
       (effects (font (size 1.27 1.27)) hide)
     )
-    (property "Datasheet" "" (id 3) (at 68.58 86.36 0)
+    (property "Datasheet" "" (id 3) (at 90.17 94.615 0)
       (effects (font (size 1.27 1.27)) hide)
     )
@@
       (reference "IC2") (unit 3) (value "74LS74") (footprint "Package_DIP:DIP-14_W7.62mm_Socket")
     )
+    (path "/790c8d76-ae9e-44ee-bffb-86dd279013aa"
+      (reference "IC5") (unit 1) (value "74LS14") (footprint "Package_DIP:DIP-14_W7.62mm_Socket")
+    )
     (path "/b0bcb598-1866-4242-9e5e-70ce53c11d1e"
