File: no-rom/vortex-f1-d-no-rom.kicad_pcb (KiCad board)
At the start: 2 copper layers, 111.9 x 64.1 mm, 47 parts, among them IC1 74LS136, IC10 uPD765AC, IC11 74HCT688, IC12 74LS38, IC13 74LS07, IC14 74LS139, IC15 74HCT688, IC2 74LS74, IC5 74LS14, IC6 74LS08, IC7 74HCT688, IC8 74LS32, IC9 FDC_9229, X1 8Mhz

Commit message: v1.0 sent to jlcpcb for production
Parts:
- added JP1: ~, Jumper:SolderJumper-3_P1.3mm_Bridged12_RoundedPad1.0x1.5mm, B.Cu at (122.0, 117.3)
- added JP2: SolderJumper_3_Bridged12, Jumper:SolderJumper-3_P1.3mm_Bridged12_RoundedPad1.0x1.5mm, B.Cu at (122.0, 114.6)
- moved R9 1.86 mm to (174.6, 115.8)
- moved C12 0.17 mm to (172.1, 115.8)
Connections:
- IC15 pad 11: +5V -> Net-(IC15-P4)
- IC15 pad 4: GND -> Net-(IC15-P1)
Routing:
- net GND: track 142.6 -> 2.54 mm, vias 63 -> 52
- net Net-(IC15-P1): track 0.00 -> 27.0 mm, vias 0 -> 1
- net Net-(IC15-P4): track 0.00 -> 11.8 mm, vias 0 -> 1
- net +5V: track 646.3 -> 643.2 mm, vias 28 -> 26
- net /D3: track 59.0 -> 62.0 mm
- net DSKD: track 94.6 -> 97.4 mm
- net ~{RDY}: track 77.0 -> 79.6 mm
- net Net-(IC10-WDATA): track 47.4 -> 49.8 mm
- net D0: track 100.5 -> 98.0 mm, vias 2 -> 1
- net /A4: track 34.1 -> 36.0 mm
- net WDOUT: track 59.0 -> 60.9 mm
- net ~{IOWR}: track 58.3 -> 60.0 mm
- net Net-(IC5-Pad1): track 22.9 -> 24.6 mm
- net WE: track 38.9 -> 40.6 mm
- net Net-(IC2A-C): track 55.5 -> 57.2 mm
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- added copper zone on B.Cu, net GND
Other:
- board text added: "Amstrad Vortex"
- board text added: "CPC-FDC v1.0"
- board text removed: "CPC-FDC v0.2"
