File: no-rom/vortex-f1-d-no-rom.kicad_sch (KiCad schematic)
At the start: 47 parts, among them IC1 74LS136, IC10 uPD765AC, IC11 74HCT688, IC12 74LS38, IC13 74LS07, IC14 74LS139, IC15 74HCT688, IC2 74LS74, IC5 74LS14, IC6 74LS08, IC7 74HCT688, IC8 74LS32, IC9 FDC_9229, X1 8Mhz

Commit message: reorganize and fix no-rom pcb and schematic
Parts:
- added unit 2 of IC8
Connections:
- net +5V: now also IC15.11 (P4); no longer IC15.4 (P1)
- net GND: now also IC15.4 (P1); no longer IC15.11 (P4)
- net ~{DS0}: now also S2.10 (Pin_10); no longer S2.26 (Pin_26)
- net ~{DS1}: now also S2.12 (Pin_12); no longer S2.24 (Pin_24)
- net ~{DS2}: now also S2.14 (Pin_14); no longer S2.22 (Pin_22)
- net ~{DS3}: now also S2.6 (Pin_6); no longer S2.30 (Pin_30)
- net ~{INDEX}: now also S2.8 (Pin_8); no longer S2.28 (Pin_28)
- net ~{IOWR}: now also IC8.5
- net ~{MOTCS}: now also IC8.4; no longer IC5.1
- net ~{MTRON}: now also S2.16 (Pin_16); no longer S2.20 (Pin_20)
- net ~{RDATA}: now also S2.30 (Pin_30); no longer S2.6 (Pin_6)
- net ~{RDY}: now also S2.34 (Pin_34); no longer S2.2 (Pin_2)
- net ~{SIDE1}: now also S2.32 (Pin_32); no longer S2.4 (Pin_4)
- net ~{STEP}: now also S2.20 (Pin_20); no longer S2.16 (Pin_16)
- net ~{TRK00}: now also S2.26 (Pin_26); no longer S2.10 (Pin_10)
- net ~{WDATA}: now also S2.22 (Pin_22); no longer S2.14 (Pin_14)
- net ~{WGATE}: now also S2.24 (Pin_24); no longer S2.12 (Pin_12)
- net ~{WPT}: now also S2.28 (Pin_28); no longer S2.8 (Pin_8)
- new net: IC5.1, IC8.6
Other:
- moved on the sheet: IC2A, IC5A

Commit message: v1.0 sent to jlcpcb for production
Parts:
- added JP1: ~, Jumper:SolderJumper-3_P1.3mm_Bridged12_RoundedPad1.0x1.5mm, symbol Jumper:SolderJumper_3_Bridged12
- added JP2: SolderJumper_3_Bridged12, Jumper:SolderJumper-3_P1.3mm_Bridged12_RoundedPad1.0x1.5mm, symbol Jumper:SolderJumper_3_Bridged12
Connections:
- net +5V: now also JP1.3 (B), JP2.1 (A); no longer IC15.11 (P4)
- net GND: now also JP1.1 (A), JP2.3 (B); no longer IC15.4 (P1)
- new net: IC15.11 (P4), JP1.2 (C)
- new net: IC15.4 (P1), JP2.2 (C)
Other:
- note added: "I/O Port Usage: &FA7E Motor Status Data Vortex: &FBF6 &FBF7 Amstrad: &FB7E &FB7F"
- note added: "JP1 and JP2 select between Vortex (default) and Amstrad FDC addresses."
- note removed: "I/O Port Usage: &FBF6 Status &FBF7 Data &FA7E Motor"
- company: (none) -> Version 1.0
- moved on the sheet: IC11, IC15, IC2A, IC5A, IC5C, IC7, IC8A, IC8B, IC8D
