File: rom-cpld/vortex-f1-d-cpld.kicad_sch (KiCad schematic)
At the start: 47 parts, among them J1 JTAG, U1 FDC 9229, U2 XC9572XL, U3 AZ1117-3.3, U4 uPD765AC, U5 AM29F010, U6 74LS06N, U7 SN74LS07N, U8 74LS06N, X1 8Mhz

Commit message: Save work
Parts:
- removed JP1: ~{VORTEX}/CPC, Jumper:SolderJumper-2_P1.3mm_Open_RoundedPad1.0x1.5mm, symbol Jumper:SolderJumper_2_Open
- added R21: 680, Resistor_SMD:R_0603_1608Metric_Pad0.98x0.95mm_HandSolder, symbol Device:R_Small
- added SW1: SW_DIP_x04, Button_Switch_THT:SW_DIP_SPSTx04_Slide_6.7x11.72mm_W7.62mm_P2.54mm_LowProfile, symbol Switch:SW_DIP_x04
Connections:
- net +5V: now also R21.2
- net A0: now also U2.45 (P45); no longer U2.33 (P33)
- net A1: now also U2.44 (P44); no longer U2.34 (P34)
- net A10: now also U2.35 (P35); no longer U2.43 (P43)
- net A13: now also U2.34 (P34); no longer U2.44 (P44)
- net A15: now also U2.33 (P33); no longer U2.45 (P45)
- net A2: now also U2.43 (P43); no longer U2.35 (P35)
- net A3: now also U2.42 (P42); no longer U2.36 (P36)
- net A4: now also U2.40 (P40); no longer U2.38 (P38)
- net A6: now also U2.38 (P38); no longer U2.40 (P40)
- net A7: now also U2.36 (P36); no longer U2.42 (P42)
- net GND: now also SW1.1, SW1.2, SW1.3, SW1.4
- net RDY: now also R21.1
- net SW1: now reaches U2.12 (P12)
- net SW1: now also SW1.8
- net SW2: now reaches U2.13 (P13)
- net SW2: now also SW1.7
- net SW4: now reaches U2.19 (P19)
- net SW4: now also SW1.5
- net ~{VORTEX}/CPC renamed SW3
- net SW3: now also SW1.6
- no-connect marks 10 -> 7

Commit message: Save CPLD work
Parts:
- removed C10, C11, C9: 100n, Capacitor_SMD:C_0603_1608Metric_Pad1.08x0.95mm_HandSolder, symbol Device:C_Small
- removed R10, R11, R12, R7, R8, R9: 10k, Resistor_SMD:R_0603_1608Metric_Pad0.98x0.95mm_HandSolder, symbol Device:R_Small
- removed R13, R14, R15, R16, R17, R18, R19, R20, R21: 680, Resistor_SMD:R_0603_1608Metric_Pad0.98x0.95mm_HandSolder, symbol Device:R_Small
- removed S2: FD Bus, Connector_IDC:IDC-Header_2x17_P2.54mm_Horizontal, symbol Connector_Generic:Conn_02x17_Odd_Even
- removed U1: FDC 9229, Package_DIP:DIP-20_W7.62mm_Socket, symbol Interface:FDC_9229
- removed U4: uPD765AC, Package_DIP:DIP-40_W15.24mm_Socket, symbol Interface:uPD765AC
- removed U6, U8: 74LS06N, Package_SO:SSOP-14_5.3x6.2mm_P0.65mm, symbol 74xx:74LS06N
- removed U7: SN74LS07N, Package_SO:SSOP-14_5.3x6.2mm_P0.65mm, symbol 74xx:SN74LS07N
- removed X1: 8Mhz, Oscillator:Oscillator_SMD_EuroQuartz_XO91-4Pin_7.0x5.0mm, symbol Oscillator:XO91
- added C13: 15pF, Capacitor_SMD:C_0603_1608Metric_Pad1.08x0.95mm_HandSolder, symbol Device:C
- added C14: 47pF, Capacitor_SMD:C_0603_1608Metric_Pad1.08x0.95mm_HandSolder, symbol Device:C
- added J2: Floppy, Connector_PinHeader_2.54mm:PinHeader_2x17_P2.54mm_Horizontal, symbol Connector_Generic:Conn_02x17_Odd_Even
- added U1: 37C65, Package_LCC:PLCC-44, symbol my_components:37C65-PLCC
- added Y1: 16MHz, Crystal:Crystal_HC49-U_Horizontal, symbol Device:Crystal_Small
- R5, R6: value 10k -> 1k
- U5: footprint Package_LCC:PLCC-32_THT-Socket -> Package_LCC:PLCC-32_11.4x14.0mm_P1.27mm
Connections:
- net +5V: no longer R2.2, R3.2, R4.2, R5.2, R6.2
- net A0: now also U1.4 (A0)
- net D0: now also U1.7 (DB0); no longer R5.1
- net D1: now also U1.8 (DB1); no longer R6.1
- net D2: now also U1.9 (DB2)
- net D3: now also U1.10 (DB3)
- net D4: now also U1.11 (DB4)
- net D5: now also U1.12 (DB5)
- net D6: now also U1.13 (DB6)
- net D7: now also U1.14 (DB7)
- net GND: now also C13.2, C14.2, J2.1 (Pin_1), J2.11 (Pin_11), J2.13 (Pin_13), J2.15 (Pin_15), J2.17 (Pin_17), J2.19 (Pin_19), J2.21 (Pin_21), J2.23 (Pin_23), J2.25 (Pin_25), J2.27 (Pin_27), J2.29 (Pin_29), J2.3 (Pin_3), J2.31 (Pin_31), J2.33 (Pin_33), J2.5 (Pin_5), J2.7 (Pin_7), J2.9 (Pin_9), U1.17 (~{DCHGEN}), U1.23 (XT2), U1.24 (DRV), U1.34 (GND)
- net RESET: now also U1.20 (RST)
- net ~{DIR}: now also J2.18 (Pin_18), U1.31 (~{DIRC})
- net ~{FDCCS}: now also U1.3 (~{CS})
- net ~{INDEX}: now also R6.1, J2.8 (Pin_8), U1.43 (~{IDX})
- net ~{IORD}: now also U1.1 (~{RD})
- net ~{IOWR}: now also U1.2 (~{WR})
- net ~{STEP}: now also J2.20 (Pin_20), U1.32 (~{STEP})
- net ~{RDATA}: now reaches R3.1
- net ~{RDATA}: now also J2.30 (Pin_30), U1.21 (~{RDD})
- net ~{DC}: now reaches R2.1
- net ~{DC}: now also J2.34 (Pin_34), U1.40 (~{DCHG})
- net ~{WP}: now reaches R4.1
- net ~{WP}: now also J2.28 (Pin_28), U1.41 (~{WP})
- new net: C13.1, U1.26 (XT1), Y1.1
- new net: C14.1, U1.25 (~{XT1}), Y1.2
- new net VCC: R2.2, R3.2, R4.2, R5.2, R6.2, U1.27 (PCVAL), U1.44 (VCC), U1.5 (~{DACK}), U1.6 (TC)
- new net ~{CCR_WR}: U1.19 (~{LDCR})
- new net ~{DENSEL}: J2.2 (Pin_2), U1.39 (~{RWC}/~{RPM})
- new net ~{DOR_WR}: U1.18 (~{LDOR})
- new net ~{DSA}: J2.14 (Pin_14), U1.33 (~{DS1})
- new net ~{DSB}: J2.12 (Pin_12), U1.35 (~{DS2})
- new net ~{HDSEL}: J2.32 (Pin_32), U1.28 (~{HS})
- new net ~{MEA}: J2.10 (Pin_10), U1.36 (~{DS3}/~{MO1})
- new net ~{MEB}: J2.16 (Pin_16), U1.37 (~{DS4}/~{MO2})
- new net ~{TRK0}: J2.26 (Pin_26), R5.1, U1.42 (~{TR00})
- new net ~{WDATA}: J2.22 (Pin_22), U1.30 (~{WD})
- new net ~{WE}: J2.24 (Pin_24), U1.29 (~{WE})
- no-connect marks 7 -> 6

Commit message: v1.0 sent to jlcpcb for production
Parts:
- removed SW1: SW_DIP_x04, Button_Switch_THT:SW_DIP_SPSTx04_Slide_6.7x11.72mm_W7.62mm_P2.54mm_LowProfile, symbol Switch:SW_DIP_x04
- Y1: footprint Crystal:Crystal_HC49-U_Horizontal -> Crystal:Crystal_SMD_7050-4Pin_7.0x5.0mm

Commit message: add new vhdl code
Parts:
- removed J1: JTAG, Connector_PinHeader_2.54mm:PinHeader_2x03_P2.54mm_Vertical, symbol Connector_Generic:Conn_02x03_Counter_Clockwise
- added J3: Micro_SD_Card, project:J_SD_Card-micro_socket_A, symbol Connector:Micro_SD_Card
- added U4: Pico, MCU_RaspberryPi_and_Boards:RPi_Pico_SMD_TH, symbol MCU_RaspberryPi_and_Boards:Pico
- R2, R3, R4, R5, R6: value 1k -> 150
Connections:
- net FLTR/STEP is gone; now on net ~{INT}: U2.2 (I/O/GTS2)
- net FLT/TRK0 is gone; now on net ~{WR}: U2.4 (P4)
- net SW1 is gone; now on net D3: U2.12 (P12)
- net SW2 is gone; now on net D4: U2.13 (P13)
- net SW3 is gone; now on net D6: U2.16 (I/O/GCK2)
- net US0 is gone; now on net ~{RD}: U2.6 (P6)
- net US1 is gone; now on net ~{IORQ}: U2.5 (I/O/GTS1)
- net WE is gone; now on net ~{M1}: U2.7 (P7)
- net ~{DS0'} is gone; now on net A8: U2.31 (P31)
- net ~{DS1'} is gone; now on net A7: U2.27 (P27)
- net ~{DS2'} is gone; now on net A6: U2.25 (P25)
- net ~{DS3'} is gone; now on net A9: U2.32 (P32)
- net ~{RW}/SEEK is gone; now on net ~{ROMEN}: U2.1 (P1)
- net +3.3V: now also J3.4 (VDD)
- net A0: now also U2.18 (P18); no longer U2.45 (P45)
- net A1: now also U2.19 (P19); no longer U2.44 (P44)
- net A10: now also U2.33 (P33); no longer U2.35 (P35)
- net A11: now also U2.34 (P34)
- net A12: now also U2.35 (P35)
- net A13: now also U2.36 (P36); no longer U2.34 (P34)
- net A14: now also U2.38 (P38)
- net A15: now also U2.39 (P39); no longer U2.33 (P33)
- net A2: now also U2.20 (P20); no longer U2.43 (P43)
- net A3: now also U2.22 (P22); no longer U2.42 (P42)
- net A4: now also U2.23 (P23); no longer U2.40 (P40)
- net A5: now also U2.24 (P24); no longer U2.39 (P39)
- net A6: no longer U2.38 (P38)
- net A7: no longer U2.36 (P36)
- net A8: no longer U2.18 (P18)
- net A9: no longer U2.17 (I/O/GCK3)
- net CLK4: no longer U2.58 (P58)
- net D0: now also U2.9 (P9), U4.21 (GPIO16); no longer U2.46 (P46)
- net D1: now also U2.10 (P10), U4.22 (GPIO17)
- net D2: now also U2.11 (P11), U4.24 (GPIO18)
- net D3: now also U4.25 (GPIO19)
- net D4: now also U4.26 (GPIO20)
- net D5: now also U2.15 (I/O/GCK1), U4.27 (GPIO21)
- net D6: now also U4.29 (GPIO22)
- net D7: now also U2.17 (I/O/GCK3), U4.31 (GPIO26_ADC0)
- net GND: now also J3.6 (VSS)
- net LED1: no longer U2.15 (I/O/GCK1)
- net MTRON: no longer U2.24 (P24)
- net READY: no longer U2.51 (P51)
- net RESET: no longer U2.8 (P8)
- net ROMA14: now also U2.64 (I/O/GSR); no longer U2.59 (P59)
- net ROMA15: now also U2.59 (P59); no longer U2.64 (I/O/GSR)
- net ROMA16: now also U2.60 (P60); no longer U2.63 (P63)
- net STEP: no longer U2.20 (P20)
- net SW4: no longer U2.19 (P19)
- net TCK: now also U4.2 (GPIO1)
- net TDI: now also U4.5 (GPIO3)
- net TDO: now also U4.4 (GPIO2)
- net TMS: now also U4.1 (GPIO0)
- net TRK00: no longer U2.23 (P23)
- net WGATE: no longer U2.22 (P22)
- net ~{FDCCS}: no longer U2.11 (P11)
- net ~{IORD}: no longer U2.9 (P9)
- net ~{IORQ}: no longer U2.48 (P48)
- net ~{IOWR}: no longer U2.10 (P10)
- net ~{MREQ}: now also U2.8 (P8); no longer U2.47 (P47)
- net ~{RD}: no longer U2.49 (P49)
- net ~{ROMEN}: no longer U2.52 (P52)
- net ~{ROMOE}: now also U2.63 (P63); no longer U2.61 (P61)
- net ~{ROMWE}: now also U2.61 (P61); no longer U2.60 (P60)
- net ~{RSET}: now also U2.52 (P52); no longer U2.56 (P56)
- net ~{WR}: no longer U2.50 (P50)
- net ~{CCR_WR} renamed ~{LDCR}
- net ~{DOR_WR} renamed ~{LDOR}
- new net PICO10: U2.45 (P45), U4.14 (GPIO10)
- new net PICO11: U2.46 (P46), U4.15 (GPIO11)
- new net PICO12: U2.44 (P44), U4.16 (GPIO12)
- new net PICO13: U2.43 (P43), U4.17 (GPIO13)
- new net PICO14: U2.42 (P42), U4.19 (GPIO14)
- new net PICO15: U2.40 (P40), U4.20 (GPIO15)
- new net SDCK: J3.5 (CLK), U4.9 (GPIO6)
- new net SDCS: J3.2 (DAT3/CD), U4.12 (GPIO9)
- new net SDDETECT: J3.9 (DETECT), U4.7 (GPIO5)
- new net SDMISO: J3.7 (DAT0), U4.11 (GPIO8)
- new net SDMOSI: J3.3 (CMD), U4.10 (GPIO7)
- no-connect marks 6 -> 23
Other:
- moved on the sheet: C13, C14, D1, J2, S1, U1, U2, U5, Y1
